Commit message: Added ati delta sensor: meshes and urdf

File: net_ft_description/urdf/net_ft_sensor_macro.urdf.xacro (robot description, xacro)
@@ -37,4 +37,13 @@
       <xacro:property name="sensor_height" value="0.0375"/>
     </xacro:if>
+    <xacro:if value="${sensor_type == 'ati_delta'}">
+      <xacro:property name="mesh_file" value="ati_delta_ft_sensor"/>
+      <xacro:property name="sensor_mass" value="0.913"/>
+      <xacro:property name="sensor_radius" value="${0.094/2}"/>
+      <xacro:property name="sensor_height" value="0.0333"/>
+      <!-- Hotfix to have correct mapping to interface type
+      in the hw interface-->
+      <xacro:property name="sensor_type" value="ati"/>
+    </xacro:if>
     <joint name="${prefix}fts_joint" type="fixed">
       <!-- The parent link must be read from the robot model it is attached to. -->
@@ -51,8 +60,8 @@
       </visual>
       <collision>
-        <origin xyz="0 0 0" rpy="0 0 0"/>
         <geometry>
-          <mesh filename="package://net_ft_description/meshes/collision/${mesh_file}.stl"/>
+          <mesh filename="package://net_ft_description/meshes/collision/${mesh_file}.stl" scale="0.001 0.001 0.001" />
         </geometry>
+	<origin xyz="${-sensor_radius} ${-sensor_radius} ${-sensor_height}" />
       </collision>
       <xacro:cylinder_inertial radius="${sensor_radius}" length="${sensor_height}" mass="${sensor_mass}">

Commit message: Added ati delta sensor type
Compared to humble, I changed the height because without the base plate
(how the sensor is normally mounted) the height is 28 mm and not 33.3
mm. For the future, fix the mesh itself removing the plate

File: net_ft_description/urdf/net_ft_sensor_macro.urdf.xacro (robot description, xacro)
@@ -37,4 +37,13 @@
       <xacro:property name="sensor_height" value="0.0375"/>
     </xacro:if>
+    <xacro:if value="${sensor_type == 'ati_delta'}">
+      <xacro:property name="mesh_file" value="ati_delta_ft_sensor"/>
+      <xacro:property name="sensor_mass" value="0.913"/>
+      <xacro:property name="sensor_radius" value="${0.094/2}"/>
+      <xacro:property name="sensor_height" value="0.028"/>
+      <!-- Hotfix to have correct mapping to interface type
+      in the hw interface-->
+      <xacro:property name="sensor_type" value="ati"/>
+    </xacro:if>
     <joint name="${prefix}fts_joint" type="fixed">
       <!-- The parent link must be read from the robot model it is attached to. -->
@@ -51,8 +60,9 @@
       </visual>
       <collision>
-        <origin xyz="0 0 0" rpy="0 0 0"/>
+	      <origin xyz="${-sensor_radius} ${-sensor_radius} ${-sensor_height}" />
         <geometry>
-          <mesh filename="package://net_ft_description/meshes/collision/${mesh_file}.stl"/>
+          <mesh filename="package://net_ft_description/meshes/collision/${mesh_file}.stl" scale="0.001 0.001 0.001" />
         </geometry>
+	      <origin xyz="${-sensor_radius} ${-sensor_radius} ${-sensor_height}" />
       </collision>
       <xacro:cylinder_inertial radius="${sensor_radius}" length="${sensor_height}" mass="${sensor_mass}">
